Commit message: frames update

File: urdf/drone.urdf.xacro (robot description, xacro)
@@ -12,5 +12,5 @@
   <!-- Horizontal LiDAR -->
   <joint name="horizontal_lidar_joint" type="fixed">
-    <origin xyz="0.2 0 0.1" rpy="0 0 0"/> <!-- Adjust position and orientation -->
+    <origin xyz="0.0 -0.07 -0.04" rpy="0 1.5708 0"/> <!-- Adjust position and orientation -->
     <parent link="base_link"/>
     <child link="horizontal_lidar_link"/>
@@ -26,5 +26,5 @@
   <!-- Vertical LiDAR -->
   <joint name="vertical_lidar_joint" type="fixed">
-    <origin xyz="-0.2 0 0.1" rpy="0 1.5708 0"/> <!-- Adjust position and orientation -->
+    <origin xyz="0.0 0.07 -0.192" rpy="0 3.14159 0"/> <!-- Adjust position and orientation -->
     <parent link="base_link"/>
     <child link="vertical_lidar_link"/>
@@ -51,5 +51,5 @@
       <child link="base_link"/>
       <origin
-        xyz="-0.12 0.0 -0.25"
+        xyz="0.0 0.0 0.0"
         rpy="0 0 0"
       />

Commit message: frame info

File: urdf/drone.urdf.xacro (robot description, xacro)
@@ -12,5 +12,5 @@
   <!-- Horizontal LiDAR -->
   <joint name="horizontal_lidar_joint" type="fixed">
-    <origin xyz="0.0 -0.07 -0.04" rpy="0 1.5708 0"/> <!-- Adjust position and orientation -->
+    <origin xyz="0.0 -0.07 -0.04" rpy="1.5708 0 0"/> <!-- Adjust position and orientation -->
     <parent link="base_link"/>
     <child link="horizontal_lidar_link"/>
@@ -26,5 +26,5 @@
   <!-- Vertical LiDAR -->
   <joint name="vertical_lidar_joint" type="fixed">
-    <origin xyz="0.0 0.07 -0.192" rpy="0 3.14159 0"/> <!-- Adjust position and orientation -->
+    <origin xyz="0.0 0.07 -0.192" rpy="3.14159 0 0"/> <!-- Adjust position and orientation -->
     <parent link="base_link"/>
     <child link="vertical_lidar_link"/>
@@ -51,5 +51,5 @@
       <child link="base_link"/>
       <origin
-        xyz="-0.12 0.0 0.25"
+        xyz="0.0 0.0 0.0"
         rpy="0 0 0"
       />

Commit message: frame info

File: urdf/drone.urdf.xacro (robot description, xacro)
@@ -1,4 +1,5 @@
 <?xml version="1.0"?>
 <robot xmlns:xacro="http://www.ros.org/wiki/xacro" name="evoii_drone">
+  <!--default values are in meters and radians-->
   <!-- Basic Drone Structure -->
   <link name="base_link">
@@ -12,5 +13,5 @@
   <!-- Horizontal LiDAR -->
   <joint name="horizontal_lidar_joint" type="fixed">
-    <origin xyz="0.0 -0.07 -0.04" rpy="1.5708 0 0"/> <!-- Adjust position and orientation -->
+    <origin xyz="-0.04 0.00 0.07" rpy="0 0 0"/> <!-- Adjust position and orientation -->
     <parent link="base_link"/>
     <child link="horizontal_lidar_link"/>
@@ -26,5 +27,5 @@
   <!-- Vertical LiDAR -->
   <joint name="vertical_lidar_joint" type="fixed">
-    <origin xyz="0.0 0.07 -0.192" rpy="3.14159 0 0"/> <!-- Adjust position and orientation -->
+    <origin xyz="-0.192 0 -0.07" rpy="0 1.507 0"/> <!-- Adjust position and orientation -->
     <parent link="base_link"/>
     <child link="vertical_lidar_link"/>

Commit message: cartographer_added

File: urdf/drone.urdf.xacro (robot description, xacro)
@@ -15,7 +15,7 @@
     <origin xyz="-0.04 0.00 0.07" rpy="0 0 0"/> <!-- Adjust position and orientation -->
     <parent link="base_link"/>
-    <child link="horizontal_lidar_link"/>
+    <child link="horizontal_laser_link"/>
   </joint>
-  <link name="horizontal_lidar_link">
+  <link name="horizontal_laser_link">
     <visual>
       <geometry>
@@ -29,7 +29,7 @@
     <origin xyz="-0.192 0 -0.07" rpy="0 1.507 0"/> <!-- Adjust position and orientation -->
     <parent link="base_link"/>
-    <child link="vertical_lidar_link"/>
+    <child link="vertical_laser_link"/>
   </joint>
-  <link name="vertical_lidar_link">
+  <link name="vertical_laser_link">
     <visual>
       <geometry>

Commit message: config change

File: urdf/drone.urdf.xacro (robot description, xacro)
@@ -2,4 +2,33 @@
 <robot xmlns:xacro="http://www.ros.org/wiki/xacro" name="evoii_drone">
   <!--default values are in meters and radians-->
+  <!-- ZED Mini Camera -->
+  <xacro:arg name="camera_name"   default="zed" />
+  <xacro:arg name="camera_model"  default="zedm" />
+  <xacro:arg name="use_zed_localization" default="true" />
+  <xacro:include filename="$(find zed_wrapper)/urdf/zed_macro.urdf.xacro" />
+  <xacro:zed_camera name="$(arg camera_name)" model="$(arg camera_model)" />
+  <!-- Add a joint to connect the ZED Camera to the robot -->
+  <xacro:if value="$(arg use_zed_localization)">
+    <!-- ZED Localization -> The reference link is '$(arg camera_name)_camera_link' and 'base_link' is a child -->
+    <joint name="$(arg camera_name)_joint" type="fixed">
+      <parent link="$(arg camera_name)_camera_link"/>
+      <child link="base_link"/>
+      <origin
+        xyz="0.0 0.0 0.0"
+        rpy="0 0 0"
+      />
+    </joint>
+  </xacro:if>
+  <xacro:unless value="$(arg use_zed_localization)">
+    <!-- NO ZED Localization -> '$(arg camera_name)_camera_link' is a child of 'base_link' -->
+    <joint name="$(arg camera_name)_joint" type="fixed">
+      <parent link="base_link"/>
+      <child link="$(arg camera_name)_camera_link"/>
+      <origin
+        xyz="0.12 0.0 0.25"
+        rpy="0 0 0"
+      />
+    </joint>
+  </xacro:unless>
   <!-- Basic Drone Structure -->
   <link name="base_link">
@@ -39,33 +68,4 @@
     </visual>
   </link>
-  <!-- ZED Mini Camera -->
-  <xacro:arg name="camera_name"   default="zed" />
-  <xacro:arg name="camera_model"  default="zedm" />
-  <xacro:arg name="use_zed_localization" default="true" />
-  <xacro:include filename="$(find zed_wrapper)/urdf/zed_macro.urdf.xacro" />
-  <xacro:zed_camera name="$(arg camera_name)" model="$(arg camera_model)" />
-  <!-- Add a joint to connect the ZED Camera to the robot -->
-  <xacro:if value="$(arg use_zed_localization)">
-    <!-- ZED Localization -> The reference link is '$(arg camera_name)_camera_link' and 'base_link' is a child -->
-    <joint name="$(arg camera_name)_joint" type="fixed">
-      <parent link="$(arg camera_name)_camera_link"/>
-      <child link="base_link"/>
-      <origin
-        xyz="0.0 0.0 0.0"
-        rpy="0 0 0"
-      />
-    </joint>
-  </xacro:if>
-  <xacro:unless value="$(arg use_zed_localization)">
-    <!-- NO ZED Localization -> '$(arg camera_name)_camera_link' is a child of 'base_link' -->
-    <joint name="$(arg camera_name)_joint" type="fixed">
-      <parent link="base_link"/>
-      <child link="$(arg camera_name)_camera_link"/>
-      <origin
-        xyz="0.12 0.0 0.25"
-        rpy="0 0 0"
-      />
-    </joint>
-  </xacro:unless>
   <!-- Materials -->
   <material name="white">

Commit message: urdf changes

File: urdf/drone.urdf.xacro (robot description, xacro)
@@ -56,5 +56,5 @@
   <!-- Vertical LiDAR -->
   <joint name="vertical_lidar_joint" type="fixed">
-    <origin xyz="-0.192 0 -0.07" rpy="0 1.507 0"/> <!-- Adjust position and orientation -->
+    <origin xyz="-0.192 0 0.005" rpy="0 1.507 0"/> <!-- Adjust position and orientation -->
     <parent link="base_link"/>
     <child link="vertical_laser_link"/>

Commit message: updated bag file record in a certain way

File: urdf/drone.urdf.xacro (robot description, xacro)
@@ -56,5 +56,5 @@
   <!-- Vertical LiDAR -->
   <joint name="vertical_lidar_joint" type="fixed">
-    <origin xyz="-0.192 0 0.005" rpy="0 1.507 0"/> <!-- Adjust position and orientation -->
+    <origin xyz="-0.192 0 0.005" rpy="0 -1.57079 0"/> <!-- Adjust position and orientation -->
     <parent link="base_link"/>
     <child link="vertical_laser_link"/>

Commit message: changed urdf

File: urdf/drone.urdf.xacro (robot description, xacro)
@@ -42,5 +42,5 @@
   <!-- Horizontal LiDAR -->
   <joint name="horizontal_lidar_joint" type="fixed">
-    <origin xyz="-0.04 0.00 0.07" rpy="0 0 0"/> <!-- Adjust position and orientation -->
+    <origin xyz="-0.04 0.00 0.07" rpy="3.141 0 0"/> <!-- Adjust position and orientation -->
     <parent link="base_link"/>
     <child link="horizontal_laser_link"/>
@@ -56,5 +56,5 @@
   <!-- Vertical LiDAR -->
   <joint name="vertical_lidar_joint" type="fixed">
-    <origin xyz="-0.192 0 0.005" rpy="0 -1.57079 0"/> <!-- Adjust position and orientation -->
+    <origin xyz="-0.192 0 0.005" rpy="3.141 -1.57079 0"/> <!-- Adjust position and orientation -->
     <parent link="base_link"/>
     <child link="vertical_laser_link"/>
